Commit message: update

File: multi_legged_controllers/urdf/spherical_joint.xacro (robot description, xacro)
@@ -26,5 +26,5 @@
       </inertial>
     </link>
-    <joint name="${name}_joint3" type="continuous">
+    <!-- <joint name="${name}_joint3" type="continuous">
       <origin rpy="0 0 0" xyz="0 0 0" />
       <parent link="${name}_junta2" />
@@ -37,8 +37,8 @@
         <inertia ixx="5.8083e-4" ixy="0" ixz="0" iyy="3.0833e-5" iyz="0" izz="5.9083e-4" />
       </inertial>
-    </link>
+    </link> -->
     <joint name="${name}_jointfixed" type="fixed">
       <origin rpy="0 0 0" xyz="0 0 -0.1" />
-      <parent link="${name}_junta3" />
+      <parent link="${name}_junta2" />
       <child link="${child}" />
     </joint>
