Commit message: t265 position update

File: multi_legged_controllers/urdf/robot_macro.xacro (robot description, xacro)
@@ -59,5 +59,5 @@
         <xacro:sensor_t265 name="${prefix}tracking_camera" topics_ns="${ns}/tracking_camera"
             parent="${prefix}base">
-            <origin xyz="0.35 0.0 0.0" rpy="0.0 -0.05 -0.0" />
+            <origin xyz="0.3 0.0 0.0" rpy="0.0 -0.05 -0.0" />
         </xacro:sensor_t265>
         <joint name="${prefix}payload_joint" type="fixed">
@@ -78,8 +78,8 @@
             </visual>
         </link>
-        <xacro:sensor_d435 name="${prefix}front_camera" topics_ns="${ns}/front_camera"
+        <!-- <xacro:sensor_d435 name="${prefix}front_camera" topics_ns="${ns}/front_camera"
             parent="${prefix}base">
             <origin xyz="0.16 0.0 0.30" rpy="0 0.54359877559 0" />
-        </xacro:sensor_d435>
+        </xacro:sensor_d435> -->
         <!-- ros_control plugin -->
         <xacro:if value="${sim}">

File: multi_legged_controllers/urdf/robot_with_prefix.xacro (robot description, xacro)
@@ -47,5 +47,5 @@
     </xacro:leg>
     <xacro:sensor_t265 name="$(arg ns)_tracking_camera" topics_ns="tracking_camera" parent="$(arg ns)_base">
-         <origin xyz="0.35 0.0 0.0" rpy="0.0 -0.05 -0.0"/>
+         <origin xyz="0.3 0.0 0.0" rpy="0.0 -0.05 -0.0"/>
     </xacro:sensor_t265>
     <joint name="$(arg ns)_payload_joint" type="fixed">

Commit message: remove payload and d435 camera

File: multi_legged_controllers/urdf/robot_macro.xacro (robot description, xacro)
@@ -68,5 +68,5 @@
         <link name="${prefix}payload">
             <inertial>
-                <mass value="3" />
+                <mass value="0.03" />
                 <origin rpy="0 0 0" xyz="0 0 0" />
                 <inertia ixx="0.025" ixy="0" ixz="0" iyy="0.021" iyz="0" izz="0.011" />

File: multi_legged_controllers/urdf/robot_with_prefix.xacro (robot description, xacro)
@@ -56,5 +56,5 @@
     <link name="$(arg ns)_payload">
         <inertial>
-            <mass value="3"/>
+            <mass value="0.03"/>
             <origin rpy="0 0 0" xyz="0 0 0"/>
             <inertia ixx="0.025" ixy="0" ixz="0" iyy="0.021" iyz="0" izz="0.011"/>
@@ -66,7 +66,7 @@
         </visual>
     </link>
-    <xacro:sensor_d435 name="$(arg ns)_front_camera" topics_ns="$(arg ns)/front_camera" parent="$(arg ns)_base">
+    <!-- <xacro:sensor_d435 name="$(arg ns)_front_camera" topics_ns="$(arg ns)/front_camera" parent="$(arg ns)_base">
            <origin xyz="0.16 0.048 0.30" rpy="0 0.54359877559 0"/>
-    </xacro:sensor_d435>
+    </xacro:sensor_d435> -->
     <xacro:if value="$(arg sim)">
     <!-- ros_control plugin -->
