Commit message: add payload

File: multi_legged_controllers/urdf/rod_with_joints_macro.xacro (robot description, xacro)
@@ -25,4 +25,31 @@
             </inertial>
         </link>
+        <joint name="payload_joint" type="fixed">
+            <parent link="rod" />
+            <child link="payload" />
+            <origin rpy="0.0 0.0 0.0" xyz="0.0 0 0.0" />
+        </joint>
+        <link name="payload">
+            <inertial>
+                <mass value="0.03" />
+                <origin rpy="0 0 0" xyz="0 0 0" />
+                <inertia ixx="0.0025" ixy="0" ixz="0" iyy="0.0021" iyz="0" izz="0.0011" />
+            </inertial>
+            <visual>
+                <origin rpy="0.0 0.0 0.0" xyz="0.0 0.0 0.0" />
+                <geometry>
+                    <box size="0.2 0.2 0.15" />
+                </geometry>
+            </visual>
+            <collision>
+                <origin rpy="0.0 0.0 0.0" xyz="0.0 0.0 0.0" />
+                <geometry>
+                    <box size="0.2 0.2 0.15" />
+                </geometry>
+            </collision>
+        </link>
+        <gazebo reference="payload">
+            <material>Gazebo/Blue</material>
+        </gazebo>
         <xacro:ball_joint name="${first_robot}_ball" parent="rod" child="${first_robot}_base">
             <origin rpy="0 0 0" xyz="0 -0.5 0" />

Commit message: update on MRA integration

File: multi_legged_controllers/urdf/rod_with_joints_macro.xacro (robot description, xacro)
@@ -32,5 +32,5 @@
         <link name="payload">
             <inertial>
-                <mass value="0.03" />
+                <mass value="5" />
                 <origin rpy="0 0 0" xyz="0 0 0" />
                 <inertia ixx="0.0025" ixy="0" ixz="0" iyy="0.0021" iyz="0" izz="0.0011" />

Commit message: Revert "add payload"
This reverts commit 4b8bce0f4a9714ff7aae2a85311a2a44ead4594d.

File: multi_legged_controllers/urdf/rod_with_joints_macro.xacro (robot description, xacro)
@@ -25,31 +25,4 @@
             </inertial>
         </link>
-        <joint name="payload_joint" type="fixed">
-            <parent link="rod" />
-            <child link="payload" />
-            <origin rpy="0.0 0.0 0.0" xyz="0.0 0 0.0" />
-        </joint>
-        <link name="payload">
-            <inertial>
-                <mass value="0.03" />
-                <origin rpy="0 0 0" xyz="0 0 0" />
-                <inertia ixx="0.0025" ixy="0" ixz="0" iyy="0.0021" iyz="0" izz="0.0011" />
-            </inertial>
-            <visual>
-                <origin rpy="0.0 0.0 0.0" xyz="0.0 0.0 0.0" />
-                <geometry>
-                    <box size="0.2 0.2 0.15" />
-                </geometry>
-            </visual>
-            <collision>
-                <origin rpy="0.0 0.0 0.0" xyz="0.0 0.0 0.0" />
-                <geometry>
-                    <box size="0.2 0.2 0.15" />
-                </geometry>
-            </collision>
-        </link>
-        <gazebo reference="payload">
-            <material>Gazebo/Blue</material>
-        </gazebo>
         <xacro:ball_joint name="${first_robot}_ball" parent="rod" child="${first_robot}_base">
             <origin rpy="0 0 0" xyz="0 -0.5 0" />
